Commit message: gazebo

File: src/differentiable-robot-model/diff_robot_data/kuka_iiwa/urdf/iiwa7.urdf (robot description, URDF)
Before this commit: robot iiwa7, 9 links, 8 joints
Links:
- added link world
Joints:
- added joint world_joint: type fixed, parent world, child iiwa_link_0, origin xyz=0.0 0.0 0.0 rpy=0.0 0.0 0.0
